File: Daylight/Disco_Daylight_on_a_stick/Daylight_Disco.kicad_pcb (KiCad board)
At the start: 2 copper layers, 270 x 11 mm, 41 parts, among them J1 Conn_01x03_Male, J2 Conn_01x03_Male, J3 Conn_01x01_Male

Commit message: Finished first version of the Daylight & Disco Sticks. Turned all leds by 90°. Rerouted tracks to be more efficient. Ordered first verison of this from jlcpcb.
Parts:
- removed the G*** at (160.0, 33.0)
- D1, D10, D11, D12, D13, D14, D15, D16, D17, D18, D2, D3, D4, D5, D6, D7, D8, D9: value WS2812B -> SK6812; footprint Daylight:LED_WS2812B_PLCC4_5.0x5.0mm_P3.2mm -> LED_SMD:LED_SK6812_PLCC4_5.0x5.0mm_P3.2mm
- moved C14 2.00 mm to (231.0, 33.0)
- moved C11 1.50 mm to (189.0, 33.0)
- moved C12 1.50 mm to (203.0, 33.0)
- moved C13 1.50 mm to (217.0, 33.0)
- moved C9 1.25 mm to (161.0, 33.0)
- moved C10 1.20 mm to (175.0, 33.0)
- moved C15 1.00 mm to (260.0, 33.0)
- moved C7 1.00 mm to (133.0, 33.0)
- moved C8 1.00 mm to (147.0, 33.0)
- moved D3 0.76 mm to (57.0, 33.0), turned to 90 degrees
- moved D16 0.76 mm to (239.0, 33.0), turned to 90 degrees
- moved D4 0.65 mm to (71.0, 33.0), turned to 90 degrees
- moved D15 0.65 mm to (225.0, 33.0), turned to 90 degrees
- moved D5 0.53 mm to (85.0, 33.0), turned to 90 degrees
- moved D14 0.53 mm to (211.0, 33.0), turned to 90 degrees
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Connections:
- D1 pad 1: +5V -> GND
- D1 pad 2: Net-(D1-Pad2) -> DIN
- D1 pad 3: GND -> +5V
- D1 pad 4: DIN -> Net-(D1-Pad4)
- D10 pad 1: +5V -> GND
- D10 pad 3: GND -> +5V
- D11 pad 1: +5V -> GND
- D11 pad 2: Net-(D11-Pad2) -> Net-(D10-Pad4)
- D11 pad 3: GND -> +5V
- D11 pad 4: Net-(D10-Pad2) -> Net-(D11-Pad4)
- D12 pad 1: +5V -> GND
- D12 pad 2: Net-(D12-Pad2) -> Net-(D11-Pad4)
- D12 pad 3: GND -> +5V
- D12 pad 4: Net-(D11-Pad2) -> Net-(D12-Pad4)
- D13 pad 1: +5V -> GND
- D13 pad 2: Net-(D13-Pad2) -> Net-(D12-Pad4)
- D13 pad 3: GND -> +5V
- D13 pad 4: Net-(D12-Pad2) -> Net-(D13-Pad4)
- D14 pad 1: +5V -> GND
- D14 pad 2: Net-(D14-Pad2) -> Net-(D13-Pad4)
- D14 pad 3: GND -> +5V
- D14 pad 4: Net-(D13-Pad2) -> Net-(D14-Pad4)
- D15 pad 1: +5V -> GND
- D15 pad 2: Net-(D15-Pad2) -> Net-(D14-Pad4)
- D15 pad 3: GND -> +5V
- D15 pad 4: Net-(D14-Pad2) -> Net-(D16-Pad2)
- D16 pad 1: +5V -> GND
- D16 pad 3: GND -> +5V
- D16 pad 4: Net-(D15-Pad2) -> Net-(D16-Pad4)
- D17 pad 1: +5V -> GND
- D17 pad 2: Net-(D17-Pad2) -> Net-(D16-Pad4)
- D17 pad 3: GND -> +5V
- D17 pad 4: Net-(D16-Pad2) -> Net-(D17-Pad4)
- D18 pad 1: +5V -> GND
- D18 pad 2: DOUT -> Net-(D17-Pad4)
- D18 pad 3: GND -> +5V
- D18 pad 4: Net-(D17-Pad2) -> DOUT
- D2 pad 1: +5V -> GND
- D2 pad 2: Net-(D2-Pad2) -> Net-(D1-Pad4)
- D2 pad 3: GND -> +5V
- D2 pad 4: Net-(D1-Pad2) -> Net-(D2-Pad4)
- D3 pad 1: +5V -> GND
- D3 pad 2: Net-(D3-Pad2) -> Net-(D2-Pad4)
- D3 pad 3: GND -> +5V
- D3 pad 4: Net-(D2-Pad2) -> Net-(D4-Pad2)
- D4 pad 1: +5V -> GND
- D4 pad 3: GND -> +5V
- D4 pad 4: Net-(D3-Pad2) -> Net-(D4-Pad4)
- D5 pad 1: +5V -> GND
- D5 pad 2: Net-(D5-Pad2) -> Net-(D4-Pad4)
- D5 pad 3: GND -> +5V
- D5 pad 4: Net-(D4-Pad2) -> Net-(D5-Pad4)
- D6 pad 1: +5V -> GND
- D6 pad 2: Net-(D6-Pad2) -> Net-(D5-Pad4)
- D6 pad 3: GND -> +5V
- D6 pad 4: Net-(D5-Pad2) -> Net-(D6-Pad4)
- D7 pad 1: +5V -> GND
- D7 pad 2: Net-(D7-Pad2) -> Net-(D6-Pad4)
- D7 pad 3: GND -> +5V
- D7 pad 4: Net-(D6-Pad2) -> Net-(D7-Pad4)
- D8 pad 1: +5V -> GND
- D8 pad 2: Net-(D8-Pad2) -> Net-(D7-Pad4)
- D8 pad 3: GND -> +5V
- D8 pad 4: Net-(D7-Pad2) -> Net-(D8-Pad4)
- D9 pad 1: +5V -> GND
- D9 pad 2: Net-(D10-Pad4) -> Net-(D8-Pad4)
- D9 pad 3: GND -> +5V
- D9 pad 4: Net-(D8-Pad2) -> Net-(D10-Pad2)
Routing:
- net Net-(D17-Pad2): track 18.0 -> 0.00 mm, vias 2 -> 0
- net Net-(D17-Pad4): track 0.00 -> 17.8 mm, vias 0 -> 2
- net Net-(D2-Pad2): track 16.5 -> 0.00 mm
- net Net-(D2-Pad4): track 0.00 -> 16.4 mm
- net Net-(D16-Pad4): track 0.00 -> 15.9 mm
- net Net-(D1-Pad4): track 0.00 -> 15.2 mm
- net Net-(D1-Pad2): track 14.0 -> 0.00 mm
- net Net-(D13-Pad4): track 0.00 -> 13.0 mm
- net Net-(D11-Pad4): track 0.00 -> 13.0 mm
- net Net-(D8-Pad4): track 0.00 -> 13.0 mm
- net Net-(D14-Pad4): track 0.00 -> 13.0 mm
- net Net-(D12-Pad4): track 0.00 -> 13.0 mm
- net Net-(D7-Pad4): track 0.00 -> 13.0 mm
- net Net-(D6-Pad4): track 0.00 -> 13.0 mm
- net Net-(D5-Pad4): track 0.00 -> 13.0 mm
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Other:
- board text added: "Daylight & Disco on a stick v1.0 by Heenne inspired by Blamm"
- board text removed: "Disco on a stick v1.1 by Blamm"
